File: sata-psu/sata-psu.kicad_sch (KiCad schematic)
At the start: 27 parts, among them Q1 20V IN, Q2 20V OUT, U1 XL4015 (5V), U2 XL4015 (12V), U5 ESP32-C3_SUPERMINI_TH, U6 ACS712xLCTR-05B, U7 ACS712xLCTR-05B

Commit message: sch: solve non-footprint erc issues
Parts:
- U1: value XL4015 (5V) -> XL4015; footprint XL4015_converter:XL4015_Converter -> (none)
- U2: value XL4015 (12V) -> XL4015
Connections:
- net GND: now also C5.2, C6.1, C7.1, C8.2, R10.1, R8.1, U6.5 (GND), U7.5 (GND)
- net +12V renamed 12V
- net +20V renamed 20V
- net +5V renamed 5V
Other:
- moved on the sheet: D3, F2, Q2

Commit message: sch: solve non-footprint erc issues
Parts:
- renumbered C7 to C1, C6 to C2, C8 to C3, C5 to C4, C2 to C5, C3 to C6, D3 to D1, D4 to D2, D2 to D3, D5 to D4, R7 to R1, R9 to R2, R8 to R3, R10 to R4, R3 to R5, R4 to R6, R5 to R7, R6 to R8, U7 to U3, U6 to U4

Commit message: wip
Parts:
- C1, C2, C3, C4: footprint (none) -> Capacitor_THT:C_Disc_D5.0mm_W2.5mm_P2.50mm
- R1, R2, R3, R4, R5, R6, R7, R8: footprint (none) -> Resistor_THT:R_Axial_DIN0207_L6.3mm_D2.5mm_P7.62mm_Horizontal
Changed lines of the file:
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@@
 		)
 		(property "Value" "GND"
-			(at 180.34 54.6099 0)
+			(at 177.8 58.42 0)
 			(show_name no)
 			(do_not_autoplace no)
@@
 					(size 1.27 1.27)
 				)
-				(justify left)
 			)
 		)
@@
 			)
 		)
-		(property "Footprint" ""
+		(property "Footprint" "Resistor_THT:R_Axial_DIN0207_L6.3mm_D2.5mm_P7.62mm_Horizontal"
 			(at 193.04 52.578 90)
 			(hide yes)
@@
 		)
 		(property "Value" "GND"
-			(at 21.59 50.7999 90)
+			(at 24.13 54.61 90)
 			(show_name no)
 			(do_not_autoplace no)
@@
 					(size 1.27 1.27)
 				)
-				(justify right)
 			)
 		)
@@
 			)
 		)
-		(property "Footprint" ""
+		(property "Footprint" "Resistor_THT:R_Axial_DIN0207_L6.3mm_D2.5mm_P7.62mm_Horizontal"
 			(at 193.04 28.448 90)
 			(hide yes)
@@
 		)
 		(property "Value" "GND"
-			(at 99.06 162.5599 0)
+			(at 96.52 166.37 0)
 			(show_name no)
 			(do_not_autoplace no)
@@
 					(size 1.27 1.27)
 				)
-				(justify left)
 			)
 		)
@@
 			)
 		)
-		(property "Footprint" ""
+		(property "Footprint" "Resistor_THT:R_Axial_DIN0207_L6.3mm_D2.5mm_P7.62mm_Horizontal"
 			(at 193.04 48.768 90)
 			(hide yes)
@@
 			)
 		)
-		(property "Footprint" ""
+		(property "Footprint" "Capacitor_THT:C_Disc_D5.0mm_W2.5mm_P2.50mm"
 			(at 133.35 47.2948 0)
 			(hide yes)
@@
 			)
 		)
-		(property "Footprint" ""
+		(property "Footprint" "Resistor_THT:R_Axial_DIN0207_L6.3mm_D2.5mm_P7.62mm_Horizontal"
 			(at 120.142 44.45 90)
 			(hide yes)
@@
 			)
 		)
-		(property "Footprint" ""
+		(property "Footprint" "Capacitor_THT:C_Disc_D5.0mm_W2.5mm_P2.50mm"
 			(at 134.62 114.6048 0)
 			(hide yes)
@@
 		)
 		(property "Footprint" "ESP32-C3_SUPERMINI_TH:MODULE_ESP32-C3_SUPERMINI_TH"
-			(at 246.38 44.45 0)
+			(at 246.38 26.67 0)
 			(hide yes)
 			(show_name no)
@@
 					(size 1.27 1.27)
 				)
-				(justify bottom)
 			)
 		)
@@
 			)
 		)
-		(property "Footprint" ""
+		(property "Footprint" "Resistor_THT:R_Axial_DIN0207_L6.3mm_D2.5mm_P7.62mm_Horizontal"
 			(at 121.412 110.49 90)
 			(hide yes)
@@
 			)
 		)
-		(property "Footprint" ""
+		(property "Footprint" "Capacitor_THT:C_Disc_D5.0mm_W2.5mm_P2.50mm"
 			(at 109.5248 60.96 0)
 			(hide yes)
@@
 			)
 		)
-		(property "Footprint" ""
+		(property "Footprint" "Resistor_THT:R_Axial_DIN0207_L6.3mm_D2.5mm_P7.62mm_Horizontal"
 			(at 129.54 35.052 90)
 			(hide yes)
@@
 			)
 		)
-		(property "Footprint" ""
+		(property "Footprint" "Capacitor_THT:C_Disc_D5.0mm_W2.5mm_P2.50mm"
 			(at 110.7948 128.27 0)
 			(hide yes)
@@
 			)
 		)
-		(property "Footprint" ""
+		(property "Footprint" "Resistor_THT:R_Axial_DIN0207_L6.3mm_D2.5mm_P7.62mm_Horizontal"
 			(at 193.04 32.258 90)
 			(hide yes)
@@
 		)
 		(property "Value" "GND"
-			(at 43.18 162.5599 0)
+			(at 40.64 166.37 0)
 			(show_name no)
 			(do_not_autoplace no)
@@
 					(size 1.27 1.27)
 				)
-				(justify left)
 			)
 		)
@@
 			)
 		)
-		(property "Footprint" ""
+		(property "Footprint" "Resistor_THT:R_Axial_DIN0207_L6.3mm_D2.5mm_P7.62mm_Horizontal"
 			(at 130.81 102.362 90)
 			(hide yes)

Commit message: wip
Parts:
- C5, C6: footprint (none) -> Capacitor_THT:CP_Radial_D10.0mm_P2.50mm_P5.00mm
- D1: footprint P6KE6V8A:DIOAD1300W80L670D310 -> Diode_THT:D_DO-15_P10.16mm_Horizontal
- D2, D3, D4: footprint P6KE16A:DIOAD1300W80L670D310 -> Diode_THT:D_DO-15_P10.16mm_Horizontal
Connections:
- net 12V: now also C2.2, U4.8 (VCC)
- net 5V: no longer C2.2, U4.8 (VCC)
Other:
- moved on the sheet: C1, C2, C3, C4, Q1, R1, R2, R3, R4, U3, U4
